File: schematics/target-panelized.kicad_pcb (KiCad board)
At the start: 2 copper layers, 200 x 214 mm, 144 parts, among them J1 Conn_01x15, J2 Conn_01x15, J4 RJ45, J5 RJ45, J8 Motor, J9 Motor, Q1 2N7002BK, Q2 2N7002BK, SW1 SW_DIP_x04, SW2 SW_DIP_x04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

Commit message: Final panelized version
Parts:
- added G***: LOGO, LOGO, B.Cu at (277.5, 159.0)
Routing:
- net Board_0-Net-(D14-K): track 54.5 -> 100.7 mm
- net Board_0-Net-(D20-K): track 164.7 -> 168.5 mm
- net Board_0-GND: vias 0 -> 1
