File: schematics/PawprintTarget.kicad_pcb (KiCad board)
At the start: 2 copper layers, 28 parts, among them J1 Screw_Terminal_01x02, J2 Screw_Terminal_01x03, J3 Screw_Terminal_01x02, J4 RJ45, J5 RJ45, J6 Screw_Terminal_01x02, J7 Screw_Terminal_01x02, Q1 IRF540N, Q2 IRF540N, SW1 SW_DIP_x04, U1 MAX485E, U2 TSOP38G36

Commit message: Component placements finished
Parts:
- removed J3, J6, J7: Screw_Terminal_01x02, Connector_Phoenix_MC:PhoenixContact_MC_1,5_2-GF-3.5_1x02_P3.50mm_Horizontal_ThreadedFlange_MountHole
- added A2: Pololu_Breakout_A4988, Module:Pololu_Breakout-16_15.2x20.3mm, B.Cu at (257.0, 104.8)
- added C4: 100uF 50V, Capacitor_SMD:CP_Elec_10x10.5, B.Cu at (268.0, 108.7)
- added D10: Enable LED, LED_SMD:LED_1206_3216Metric, F.Cu at (232.0, 123.5)
- added D11: Enable LED, LED_SMD:LED_1206_3216Metric, F.Cu at (200.1, 108.5)
- added D12: Enable LED, LED_SMD:LED_1206_3216Metric, F.Cu at (168.0, 123.5)
- added D13: Enable LED, LED_SMD:LED_1206_3216Metric, F.Cu at (158.0, 150.5)
- added D14: Enable LED, LED_SMD:LED_1206_3216Metric, F.Cu at (189.5, 150.1)
- added D15: SM712_SOT23, Package_TO_SOT_SMD:SOT-23, B.Cu at (255.6, 146.0)
- added D16: Hit LED, LED_SMD:LED_1206_3216Metric, F.Cu at (200.0, 139.0)
- added D17: Hit LED, LED_SMD:LED_1206_3216Metric, F.Cu at (200.1, 60.0)
- added D18: Hit LED, LED_SMD:LED_1206_3216Metric, F.Cu at (135.0, 88.0)
- added D19: Hit LED, LED_SMD:LED_1206_3216Metric, F.Cu at (110.2, 150.0)
- added D20: Hit LED, LED_SMD:LED_1206_3216Metric, F.Cu at (131.5, 207.5)
- added D21: Hit LED, LED_SMD:LED_1206_3216Metric, F.Cu at (268.5, 91.5)
- added D22: Hit LED, LED_SMD:LED_1206_3216Metric, F.Cu at (289.8, 150.0)
- added D23: Hit LED, LED_SMD:LED_1206_3216Metric, F.Cu at (269.6, 207.0)
- added D24: Hit LED, LED_SMD:LED_1206_3216Metric, F.Cu at (200.0, 239.8)
- added D25: Hit LED, LED_SMD:LED_1206_3216Metric, F.Cu at (200.0, 161.0)
- added D5: Enable LED, LED_SMD:LED_1206_3216Metric, F.Cu at (241.0, 150.0)
- added D6: Enable LED, LED_SMD:LED_1206_3216Metric, F.Cu at (211.0, 150.0)
- added D7: Enable LED, LED_SMD:LED_1206_3216Metric, F.Cu at (232.0, 176.5)
- added D8: Enable LED, LED_SMD:LED_1206_3216Metric, F.Cu at (200.1, 191.4)
- added D9: Enable LED, LED_SMD:LED_1206_3216Metric, F.Cu at (168.0, 176.5)
- added FID1: Fiducial, Fiducial:Fiducial_1mm_Mask2mm, F.Cu at (200.0, 245.5)
- added FID1: Fiducial, Fiducial:Fiducial_1mm_Mask2mm, B.Cu at (200.0, 245.5)
- added FID2: Fiducial, Fiducial:Fiducial_1mm_Mask2mm, F.Cu at (200.0, 54.0)
- added FID2: Fiducial, Fiducial:Fiducial_1mm_Mask2mm, B.Cu at (200.0, 54.0)
- added FID3: Fiducial, Fiducial:Fiducial_1mm_Mask2mm, F.Cu at (105.5, 150.0)
- added FID3: Fiducial, Fiducial:Fiducial_1mm_Mask2mm, B.Cu at (105.5, 150.0)
- added FID4: Fiducial, Fiducial:Fiducial_1mm_Mask2mm, F.Cu at (296.0, 150.0)
- added FID4: Fiducial, Fiducial:Fiducial_1mm_Mask2mm, B.Cu at (296.0, 150.0)
- added J8: Motor, Connector_PinSocket_2.54mm:PinSocket_1x04_P2.54mm_Vertical, B.Cu at (282.0, 126.5)
- added J9: Motor, Connector_JST:JST_PH_B4B-PH-K_1x04_P2.00mm_Vertical, B.Cu at (275.0, 127.0)
- added JP1: EtherKiller1, Jumper:SolderJumper-2_P1.3mm_Open_TrianglePad1.0x1.5mm, B.Cu at (155.5, 155.0)
- added JP2: EtherKiller2, Jumper:SolderJumper-2_P1.3mm_Open_TrianglePad1.0x1.5mm, B.Cu at (162.8, 152.5)
- added JP3: Filter Bypass, Jumper:SolderJumper-2_P1.3mm_Open_TrianglePad1.0x1.5mm, B.Cu at (152.5, 129.2)
- added R5: R, Resistor_SMD:R_0603_1608Metric, B.Cu at (232.2, 86.5)
- added REF**: MountingHole_6.4mm_M6_Pad_Via, MountingHole:MountingHole_6.4mm_M6_Pad_Via, F.Cu at (215.0, 165.0)
- added REF**: MountingHole_6.4mm_M6_Pad_Via, MountingHole:MountingHole_6.4mm_M6_Pad_Via, F.Cu at (215.0, 135.0)
- added REF**: MountingHole_6.4mm_M6_Pad_Via, MountingHole:MountingHole_6.4mm_M6_Pad_Via, F.Cu at (185.0, 135.0)
- added REF**: MountingHole_6.4mm_M6_Pad_Via, MountingHole:MountingHole_6.4mm_M6_Pad_Via, F.Cu at (185.0, 165.0)
- added SW2: SW_DIP_x04, Button_Switch_THT:SW_DIP_SPSTx04_Piano_10.8x11.72mm_W7.62mm_P2.54mm, B.Cu at (246.9, 85.4)
- added U3: Mini360, Mini360_step-down:Mini360_step-down, B.Cu at (187.9, 78.1)
- A1, J4, J5, SW1, U1: moved to B.Cu
- C1, C3: footprint Capacitor_THT:C_Disc_D3.0mm_W2.0mm_P2.50mm -> Capacitor_SMD:C_0805_2012Metric; moved to B.Cu
- C2: footprint Capacitor_THT:CP_Radial_D5.0mm_P2.00mm -> Capacitor_SMD:C_1206_3216Metric; moved to B.Cu
- D1, D2, D3, D4: footprint LED_THT:LED_D3.0mm -> LED_SMD:LED_1206_3216Metric; moved to B.Cu
- J1: value Screw_Terminal_01x02 -> Conn_01x15; footprint Connector_Phoenix_MC:PhoenixContact_MC_1,5_2-GF-3.5_1x02_P3.50mm_Horizontal_ThreadedFlange_MountHole -> Connector_PinSocket_2.54mm:PinSocket_1x15_P2.54mm_Vertical; moved to B.Cu
- J2: value Screw_Terminal_01x03 -> Conn_01x15; footprint Connector_Phoenix_MC:PhoenixContact_MC_1,5_3-G-3.5_1x03_P3.50mm_Horizontal -> Connector_PinSocket_2.54mm:PinSocket_1x15_P2.54mm_Vertical; moved to B.Cu
- L1: footprint Inductor_THT:L_Radial_D9.5mm_P5.00mm_Fastron_07HVP -> Mini360_step-down:Inductor_SDR1307; moved to B.Cu
- Q1, Q2: value IRF540N -> 2N7002BK; footprint Package_TO_SOT_THT:TO-220-3_Vertical -> Package_TO_SOT_SMD:SOT-23-3; moved to B.Cu
- R1, R2, R3, R4: value 1k -> 2k; footprint Resistor_SMD:R_1210_3225Metric -> Resistor_SMD:R_0603_1608Metric; moved to B.Cu
- R6, R7: value 200 -> R; footprint Resistor_SMD:R_1210_3225Metric -> Resistor_SMD:R_0603_1608Metric; moved to B.Cu
- R8: value DNI -> R; footprint Resistor_SMD:R_1210_3225Metric -> Resistor_SMD:R_0603_1608Metric; moved to B.Cu
- U2: value TSOP38G36 -> EAIRMCA1; footprint OptoDevice:Vishay_MINICAST-3Pin -> OptoDevice:Vishay_MOLD-3Pin; moved to B.Cu
- moved SW1 178.4 mm to (237.5, 209.1)
- moved J4 166.9 mm to (268.9, 146.0), turned to -90 degrees
- moved R6 156.7 mm to (232.2, 83.0)
- moved R7 156.0 mm to (232.0, 94.0)
- moved U1 154.7 mm to (241.1, 139.5), turned to 0 degrees
- moved R8 136.7 mm to (232.2, 77.5), turned to 0 degrees
- moved A1 119.0 mm to (219.6, 114.2), turned to 90 degrees
- moved U2 104.7 mm to (206.5, 152.5)
- moved C2 95.0 mm to (153.0, 140.5)
- moved C3 85.7 mm to (175.0, 92.0)
- moved L1 85.5 mm to (152.5, 129.4), turned to 180 degrees
- moved Q2 85.3 mm to (166.4, 108.5), turned to 180 degrees
- moved C1 76.6 mm to (153.1, 119.0), turned to 0 degrees
- moved D1 70.6 mm to (121.1, 135.0)
- moved R1 70.1 mm to (131.0, 135.0)
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Connections:
- A1 pad 10: LGHTS2 -> DIR
- A1 pad 11: Net-(A1-D8) -> D8
- A1 pad 12: unconnected-(A1-D9-Pad12) -> D9
- A1 pad 13: Net-(A1-D10) -> D10
- A1 pad 14: Net-(A1-MOSI) -> MOSI
- A1 pad 15: Net-(A1-MISO) -> MISO
- A1 pad 16: unconnected-(A1-SCK-Pad16) -> SCK
- A1 pad 17: unconnected-(A1-3V3-Pad17) -> +3.3V
- A1 pad 18: unconnected-(A1-AREF-Pad18) -> AREF
- A1 pad 19: unconnected-(A1-A0-Pad19) -> IR_Signal
- A1 pad 20: unconnected-(A1-A1-Pad20) -> A1
- A1 pad 21: unconnected-(A1-A2-Pad21) -> A2
- A1 pad 22: unconnected-(A1-A3-Pad22) -> A3
- A1 pad 23: unconnected-(A1-SDA/A4-Pad23) -> SDA/A4
- A1 pad 24: unconnected-(A1-SCL/A5-Pad24) -> SCL/A5
- A1 pad 25: unconnected-(A1-A6-Pad25) -> A6
- A1 pad 26: IR_Signal -> A7
- A1 pad 28: unconnected-(A1-~{RESET}-Pad28) -> RESET2
- A1 pad 29: GND -> RJ45_7
- A1 pad 3: unconnected-(A1-~{RESET}-Pad3) -> RESET
- A1 pad 30: +12V -> MCU VIN
- A1 pad 4: GND -> RJ45_7
- A1 pad 9: LGHTS1 -> STEP
- C1 pad 1: PWR IN -> RJ45_8
- C1 pad 2: GND -> RJ45_7
- C2 pad 1: +12V -> +24V
- C2 pad 2: GND -> RJ45_7
- C3 pad 2: GND -> RJ45_7
- D1 pad 1: GND -> RJ45_7
- D2 pad 1: GND -> RJ45_7
- D3 pad 1: GND -> RJ45_7
- D4 pad 1: GND -> RJ45_7
- J1 pad 1: SignalA -> Driver_Input
- J1 pad 2: SignalB -> Receiver_Output
- J2 pad 1: PWR IN -> SCK
- J2 pad 2: EnableRJ45 -> +3.3V
- J2 pad 3: HitRJ45 -> AREF
- J4 pad 1: GND -> RJ45_7
- J4 pad 2: EnableRJ45 -> RJ45_7
- J4 pad 3: HitRJ45 -> SignalB
- J4 pad 4: GND -> RJ45_8
- J4 pad 5: SignalB -> RJ45_8
- J4 pad 7: GND -> Net-(JP1-A)
- J4 pad 8: PWR IN -> Net-(JP2-A)
- J5 pad 1: GND -> RJ45_7
- J5 pad 2: EnableRJ45 -> RJ45_7
- J5 pad 3: HitRJ45 -> SignalB
- J5 pad 4: GND -> RJ45_8
- J5 pad 5: SignalB -> RJ45_8
- J5 pad 7: GND -> RJ45_7
- J5 pad 8: PWR IN -> RJ45_8
- L1 pad 1: PWR IN -> RJ45_8
- L1 pad 2: +12V -> +24V
- Q1 pad 1: Hit_Indicator -> unconnected-(Q1-G-Pad1)
- Q1 pad 2: HitRJ45 -> Net-(D20-K)
- Q1 pad 3: GND -> RJ45_7
- Q2 pad 2: EnableRJ45 -> Net-(D14-K)
- Q2 pad 3: GND -> RJ45_7
- R1 pad 2: +12V -> +24V
- R6 pad 1: Net-(J6-Pin_2) -> +24V
- R6 pad 2: LGHTS1 -> Net-(D10-A)
- R7 pad 1: Net-(J7-Pin_2) -> +24V
- R7 pad 2: LGHTS2 -> Net-(D16-A)
- R8 pad 1: SignalB -> +24V
- R8 pad 2: SignalA -> Net-(D21-A)
- SW1 pad 1: GND -> RJ45_7
- SW1 pad 2: GND -> RJ45_7
- SW1 pad 3: GND -> RJ45_7
- SW1 pad 4: GND -> RJ45_7
- SW1 pad 5: Net-(A1-MISO) -> D8
- SW1 pad 6: Net-(A1-MOSI) -> D9
- SW1 pad 7: Net-(A1-D10) -> D10
- SW1 pad 8: Net-(A1-D8) -> MOSI
- U1 pad 5: GND -> RJ45_7
- U2 pad 2: GND -> RJ45_7
Other:
- board outline added: 200 x 200 mm
- board text added: "Mounting: M6, 35mm center-to-center square Board diameter: 200mm"
- board text added: "V"

Commit message: Fix RJ45 connector
Parts:
- moved JP2 10.5 mm to (153.3, 148.0), turned to 0 degrees
- moved JP1 0.72 mm to (154.8, 155.0), turned to -90 degrees
- turned D17 to 0 degrees
Connections:
- A1 pad 29: RJ45_7 -> GND
- A1 pad 4: RJ45_7 -> GND
- A2 pad 1: RJ45_7 -> GND
- A2 pad 13: RJ45_7 -> GND
- A2 pad 14: RJ45_7 -> GND
- A2 pad 7: RJ45_7 -> GND
- A2 pad 8: RJ45_8 -> +VDC
- A2 pad 9: RJ45_7 -> GND
- C1 pad 1: RJ45_8 -> +VDC
- C1 pad 2: RJ45_7 -> GND
- C2 pad 2: RJ45_7 -> GND
- C3 pad 2: RJ45_7 -> GND
- C4 pad 1: RJ45_8 -> +VDC
- C4 pad 2: RJ45_7 -> GND
- D1 pad 1: RJ45_7 -> GND
- D15 pad 3: RJ45_7 -> GND
- D2 pad 1: RJ45_7 -> GND
- D3 pad 1: RJ45_7 -> GND
- D4 pad 1: RJ45_7 -> GND
- J1 pad 4: RJ45_7 -> GND
- J2 pad 14: RJ45_7 -> GND
- J4 pad 1: RJ45_7 -> GND
- J4 pad 2: RJ45_7 -> GND
- J4 pad 4: RJ45_8 -> +VDC
- J4 pad 5: RJ45_8 -> +VDC
- J4 pad 7: Net-(JP1-A) -> RJ45_7
- J4 pad 8: Net-(JP2-A) -> RJ45_8
- J5 pad 1: RJ45_7 -> GND
- J5 pad 2: RJ45_7 -> GND
- J5 pad 4: RJ45_8 -> +VDC
- J5 pad 5: RJ45_8 -> +VDC
- JP1 pad 1: Net-(JP1-A) -> RJ45_7
- JP1 pad 2: RJ45_7 -> GND
- JP2 pad 1: Net-(JP2-A) -> RJ45_8
- JP2 pad 2: RJ45_8 -> +VDC
- JP3 pad 1: RJ45_8 -> +VDC
- L1 pad 1: RJ45_8 -> +VDC
- Q1 pad 3: RJ45_7 -> GND
- Q2 pad 3: RJ45_7 -> GND
- SW1 pad 1: RJ45_7 -> GND
- SW1 pad 2: RJ45_7 -> GND
- SW1 pad 3: RJ45_7 -> GND
- SW1 pad 4: RJ45_7 -> GND
- U1 pad 5: RJ45_7 -> GND
- U2 pad 2: RJ45_7 -> GND
- U3 pad 1: RJ45_7 -> GND
- U3 pad 3: RJ45_7 -> GND
Routing:
- net RJ45_7: track 0.00 -> 183.2 mm
- net +5V: track 0.00 -> 88.3 mm
- net Net-(D23-K): track 0.00 -> 80.4 mm
- net Net-(D24-K): track 0.00 -> 78.3 mm
- net Net-(D17-K): track 0.00 -> 73.9 mm
- net Net-(D18-K): track 0.00 -> 69.5 mm
- net IR_Signal: track 0.00 -> 65.7 mm
- net Net-(D21-K): track 0.00 -> 64.5 mm
- net Net-(D19-K): track 0.00 -> 63.5 mm
- net Net-(D22-K): track 0.00 -> 62.6 mm
- net DIR: track 0.00 -> 56.8 mm
- net STEP: track 0.00 -> 53.2 mm
- net SignalB: track 0.00 -> 28.8 mm
- net Net-(A2-MS3): track 0.00 -> 25.1 mm
- net +VDC: track 0.00 -> 17.6 mm
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
Commit message: Done, probably
- Nicer labels
- Probably won't blow up
Parts:
- moved C3 87.4 mm to (245.0, 144.4), turned to 0 degrees
- moved C2 21.5 mm to (152.3, 119.0)
- moved C1 20.6 mm to (152.5, 139.6), turned to 180 degrees
- moved JP1 5.83 mm to (155.4, 160.8)
- moved FID3 2.90 mm to (102.6, 150.0) (x2)
- moved FID1 2.10 mm to (200.0, 247.6) (x2)
- moved FID4 1.60 mm to (297.6, 150.0) (x2)
- moved FID2 1.20 mm to (200.0, 52.8) (x2)
- moved R7 0.18 mm to (232.2, 94.0)
- turned JP3 to 90 degrees
- turned L1 to 0 degrees
Connections:
- Q1 pad 1: unconnected-(Q1-G-Pad1) -> Hit_Indicator
Routing:
- net +VDC: track 17.6 -> 209.8 mm, vias 0 -> 3
- net SignalA: track 13.6 -> 189.3 mm, vias 0 -> 1
- net Net-(D20-K): track 0.00 -> 164.7 mm, vias 0 -> 1
- net SignalB: track 28.8 -> 188.7 mm
- net +24V: track 0.00 -> 145.4 mm, vias 0 -> 1
- net RJ45_8: track 10.8 -> 153.4 mm
- net MOSI: track 5.29 -> 137.3 mm, vias 0 -> 1
- net D10: track 5.29 -> 126.5 mm, vias 0 -> 1
- net D9: track 5.29 -> 125.3 mm, vias 0 -> 1
- net Hit_Indicator: track 5.29 -> 125.0 mm, vias 0 -> 2
- net +5V: track 88.3 -> 197.9 mm, vias 0 -> 1
- net D8: track 5.29 -> 110.3 mm
- net Enable_Indicator: track 5.29 -> 98.1 mm
- net Net-(D16-K): track 0.00 -> 81.8 mm
- net IR_Signal: track 65.7 -> 145.2 mm
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- added copper zone on B.Cu, net GND
- added copper zone on F.Cu, net GND
Other:
- board text added: "1-2: GND 3: RS485+ (A) 4-6: 24V+ 6: RS485- (B) 7: GND (OPT) 8: 24V+ (OPT)"
- board text added: "5V+"
- board text added: "Bridge JP1 & JP2 if you aren't afraid to kill Ethernet devices"
- board text added: "GND"
- board text added: "Mini360"
- board text added: "Pawprint Prototyping OpenSauce 2025 A.R.M. Target Controller rev A"
- board text added: "VIN"
- board text added: "v"

Commit message: Final panelized version
Routing:
- net Net-(D14-K): track 54.5 -> 96.7 mm
- net Net-(D20-K): track 164.7 -> 167.0 mm
- net GND: vias 0 -> 1
Changed lines of the file:
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@@
+	)
+	(segment
+		(start 190.676 149.876)
+		(end 189.5 148.7)
+		(width 0.2)
+		(layer "F.Cu")
+		(net 56)
 	)
 	(segment
@@
 		(start 189.223354 148.7)
 		(end 178.299 137.775646)
+		(width 0.2)
+		(layer "F.Cu")
+		(net 56)
+	)
+	(segment
+		(start 190.36016 152.426)
+		(end 190.676 152.11016)
+		(width 0.2)
+		(layer "F.Cu")
+		(net 56)
+	)
+	(segment
+		(start 167.020102 166.979898)
+		(end 181.574 152.426)
+		(width 0.2)
+		(layer "F.Cu")
+		(net 56)
+	)
+	(segment
+		(start 190.676 152.11016)
+		(end 190.676 149.876)
+		(width 0.2)
+		(layer "F.Cu")
+		(net 56)
+	)
+	(segment
+		(start 167.020102 175.520102)
+		(end 167.020102 166.979898)
+		(width 0.2)
+		(layer "F.Cu")
+		(net 56)
+	)
+	(segment
+		(start 181.574 152.426)
+		(end 190.36016 152.426)
 		(width 0.2)
 		(layer "F.Cu")
@@
 	)
 	(segment
-		(start 187.899 171.701)
-		(end 198.6 161)
-		(width 0.2)
-		(layer "F.Cu")
-		(net 63)
-	)
-	(segment
 		(start 192.2 154.6)
 		(end 192.2 132.723354)
@@
 	)
 	(segment
-		(start 132.5 208.5)
-		(end 169.299 171.701)
-		(width 0.2)
-		(layer "F.Cu")
-		(net 63)
-	)
-	(segment
-		(start 169.299 171.701)
-		(end 187.899 171.701)
+		(start 189 174.5)
+		(end 170 174.5)
+		(width 0.2)
+		(layer "F.Cu")
+		(net 63)
+	)
+	(segment
+		(start 136 208.5)
+		(end 132.5 208.5)
 		(width 0.2)
 		(layer "F.Cu")
@@
 	)
 	(segment
+		(start 170 174.5)
+		(end 136 208.5)
+		(width 0.2)
+		(layer "F.Cu")
+		(net 63)
+	)
+	(segment
 		(start 192.2 132.723354)
 		(end 185.291 125.814354)
+		(width 0.2)
+		(layer "F.Cu")
+		(net 63)
+	)
+	(segment
+		(start 198.6 161)
+		(end 198.6 164.9)
+		(width 0.2)
+		(layer "F.Cu")
+		(net 63)
+	)
+	(segment
+		(start 198.6 164.9)
+		(end 189 174.5)
 		(width 0.2)
 		(layer "F.Cu")
@@
 		(net 69)
 	)
+	(via
+		(at 164.5 110.5)
+		(size 0.6)
+		(drill 0.3)
+		(layers "F.Cu" "B.Cu")
+		(free yes)
+		(net 69)
+	)

Commit message: Oh my god I'm so stupid
Parts:
- added G***: LOGO, LOGO, B.Cu at (270.5, 182.5)
- moved REF** 3.54 mm to (217.5, 167.5)
- moved REF** 3.54 mm to (217.5, 132.5)
- moved REF** 3.54 mm to (182.5, 132.5)
- moved REF** 3.54 mm to (182.5, 167.5)
Routing:
- net Net-(D14-K): track 96.7 -> 101.9 mm
- net RJ45_8: track 153.4 -> 155.8 mm
- net GND: track 6.16 -> 7.93 mm, vias 1 -> 3
- net D8: track 110.3 -> 112.1 mm
- net Net-(D6-K): track 33.8 -> 35.4 mm
- net RJ45_7: track 169.2 -> 168.7 mm
